Commit message: final version

File: urdf/birdbot_v00.urdf (robot description, URDF)
Before this commit: robot urdf_vis/birdbot, 9 links, 8 joints
Links:
- link base_link: mass 0.246924141249937 -> 0.24692; geometry collision mesh filename=package://urdf_vis/meshes/birdbot_v00/base_link.STL; visual mesh filename=package://urdf_vis/meshes/birdbot_v00/base_link.STL
- link left_femur_link: mass 0.0327221036602836 -> 0.032722; geometry collision mesh filename=package://urdf_vis/meshes/birdbot_v00/left_femur_link.STL; visual mesh filename=package://urdf_vis/meshes/birdbot_v00/left_femur_link.STL
- link left_foot_link: mass 0.0101123797998784 -> 0.010112; geometry collision mesh filename=package://urdf_vis/meshes/birdbot_v00/left_foot_link.STL; visual mesh filename=package://urdf_vis/meshes/birdbot_v00/left_foot_link.STL
- link left_pelvis_link: mass 0.0240397099024521 -> 0.02404; geometry collision mesh filename=package://urdf_vis/meshes/birdbot_v00/left_pelvis_link.STL; visual mesh filename=package://urdf_vis/meshes/birdbot_v00/left_pelvis_link.STL
- link left_tibia_link: mass 0.0179012857998286 -> 0.017901; geometry collision mesh filename=package://urdf_vis/meshes/birdbot_v00/left_tibia_link.STL; visual mesh filename=package://urdf_vis/meshes/birdbot_v00/left_tibia_link.STL
- link right_femur_link: mass 0.0327221032031459 -> 0.0327221041849724; geometry collision mesh filename=package://urdf_vis/meshes/birdbot_v00/right_femur_link.STL; visual mesh filename=package://urdf_vis/meshes/birdbot_v00/right_femur_link.STL
- link right_foot_link: mass 0.0101123797998784 -> 0.0101123787795885; geometry collision mesh filename=package://urdf_vis/meshes/birdbot_v00/right_foot_link.STL; visual mesh filename=package://urdf_vis/meshes/birdbot_v00/right_foot_link.STL
- link right_pelvis_link: mass 0.0240397097940218 -> 0; geometry collision mesh filename=package://urdf_vis/meshes/birdbot_v00/right_pelvis_link.STL; visual mesh filename=package://urdf_vis/meshes/birdbot_v00/right_pelvis_link.STL
- link right_tibia_link: mass 0.0179012857998287 -> 0.0179012926659031; geometry collision mesh filename=package://urdf_vis/meshes/birdbot_v00/right_tibia_link.STL; visual mesh filename=package://urdf_vis/meshes/birdbot_v00/right_tibia_link.STL
Joints:
- joint left_femur_joint: origin xyz=0.00890000000000016 0 0.0850000000000003 rpy=-1.5707963267949 0.551803682745526 1.5707963267949 -> xyz=0.0089 0.073612 0.0425 rpy=-1.5708 1.3727 1.5708
- joint left_foot_joint: axis 0 -1 0 -> 0 0 1; origin xyz=0 0 0.105 rpy=1.5707963267949 -0.530471978203955 1.5707963267949 -> xyz=0 0.013912 0.10407 rpy=1.5708 0.066441 1.5708; type fixed -> continuous
- joint left_pelvis_joint: origin xyz=0.00121592635923147 -0.000878363870458104 0.0247999999999999 rpy=1.64268091463056 -1.5707963267949 0 -> xyz=0 -0.0248 0 rpy=-2.618 0 -1.5708
- joint left_tibia_joint: origin xyz=-0.109999587813108 -0.000301132771852231 0 rpy=1.5202434435008 1.5707963267949 0 -> xyz=-0.11 -0.00030113 0 rpy=2.4863 1.5708 0
- joint right_femur_joint: origin xyz=-0.0085499999999998 0 0.0850000000000003 rpy=-1.5707963267949 0.551803682745524 1.5707963267949 -> xyz=-0.0042882 0.073612 0.0425 rpy=-1.5708 1.3727 1.5708
- joint right_foot_joint: axis 0 -1 0 -> 0 0 1; origin xyz=0 0 0.105 rpy=1.5707963267949 -0.530471978203955 1.5707963267949 -> xyz=-0.00019997 0.013912 0.10407 rpy=1.5708 0.066441 1.5708; type fixed -> continuous
- joint right_pelvis_joint: origin xyz=0.00121592635923147 -0.000878363870458081 -0.0252000000000001 rpy=1.64268091463056 -1.5707963267949 0 -> xyz=0 0.029412 0 rpy=-2.618 0 -1.5708
- joint right_tibia_joint: origin xyz=-0.109999587813108 -0.000301132771851897 0 rpy=1.5202434435008 1.5707963267949 0 -> xyz=-0.11 -0.00030113 0 rpy=2.4863 1.5708 0
